File: schematics/skunk.sch (KiCad schematic (older format))
At the start: 37 parts

Commit message: Added arduino pins with numbers and functions
Parts:
- added P?: DIL16, symbol DIL16
Connections:
- net labels added: 31, 32, 33, 34, 35, 36, 37, 5, 53, 7, 9, A0, A1, BATT_IN, KEYSW_IN, POT_IN, R5, R6, R7, UART1 RX, UART1 TX, UART2 TX
- wire segments 166 -> 182
Changed lines of the file:
@@
-EESchema Schematic File Version 2  date Fri 05 Oct 2012 15:41:18 BST
+EESchema Schematic File Version 2  date Fri 05 Oct 2012 19:19:31 BST
 LIBS:power
 LIBS:device
@@
 	1    0    0    -1
 $EndComp
+$Comp
+L FUSE F?
+U 1 1 506F151A
+P 3800 750
+F 0 "F?" H 3900 800 40  0000 C CNN
+F 1 "FUSE 1A" H 3750 600 40  0000 C CNN
+	1    3800 750
+	1    0    0    -1
+$EndComp
+Text Label 3250 750  0    60   ~ 0
++16V
+Text Label 3300 1700 0    60   ~ 0
+0V
+$Comp
+L C C?
+U 1 1 506F1B91
+P 4150 1150
+F 0 "C?" H 4200 1250 50  0000 L CNN
+F 1 "100nF" H 4200 1050 50  0000 L CNN
+	1    4150 1150
+	1    0    0    -1
+$EndComp
+$Comp
+L ZENER D?
+U 1 1 506F1D24
+P 4600 950
+F 0 "D?" H 4600 1050 50  0000 C CNN
+F 1 "20V" H 4600 850 40  0000 C CNN
+	1    4600 950
+	0    -1   -1   0
+$EndComp
+$Comp
+L R R?
+U 1 1 506F1D33
+P 4600 1450
+F 0 "R?" V 4680 1450 50  0000 C CNN
+F 1 "1k" V 4600 1450 50  0000 C CNN
+	1    4600 1450
+	1    0    0    -1
+$EndComp
+$Comp
+L C C?
+U 1 1 506F22D9
+P 4900 1450
+F 0 "C?" H 4950 1550 50  0000 L CNN
+F 1 "47nF" H 4950 1350 50  0000 L CNN
+	1    4900 1450
+	1    0    0    -1
+$EndComp
+$Comp
+L THYRISTOR T?
+U 1 1 506F2A69
+P 5300 1100
+F 0 "T?" H 5200 1200 40  0000 C CNN
+F 1 "THYRISTOR" H 5300 1000 40  0000 C CNN
+	1    5300 1100
+	0    -1   1    0
+$EndComp
+Text Notes 1150 1750 0    60   ~ 0
+POWER INPUT\n
+Text Notes 3700 1850 0    60   ~ 0
+OVERVOLTAGE CROWBAR
+$Comp
+L DIODE D?
+U 1 1 506F2E41
+P 1650 2450
+F 0 "D?" H 1650 2550 40  0000 C CNN
+F 1 "DIODE" H 1650 2350 40  0000 C CNN
+	1    1650 2450
+	0    -1   -1   0
+$EndComp
+Text Notes 1350 2650 0    60   ~ 0
+IDIOT\nDIODE
+Text Notes 14700 1900 0    60   ~ 0
+FLOWMETER CONNECTION
+Text Notes 7450 7950 0    60   ~ 0
+PERIPHERAL CONNECTION CABLE
+Text Notes 11150 7900 0    60   ~ 0
+PERIPHERALS
 Wire Wire Line
 	9500 1250 15050 1250
@@
 	9500 1150 9200 1150
 Wire Wire Line
-	9200 750  9200 1150
+	9200 1150 9200 750
 Wire Wire Line
 	9300 1050 15050 1050
@@
 	3000 750  3550 750
 Wire Wire Line
-	4050 750  9200 750
-$Comp
-L FUSE F?
-U 1 1 506F151A
-P 3800 750
-F 0 "F?" H 3900 800 40  0000 C CNN
-F 1 "FUSE 1A" H 3750 600 40  0000 C CNN
-	1    3800 750
-	1    0    0    -1
-$EndComp
-Text Label 3250 750  0    60   ~ 0
-+16V
-Text Label 3300 1700 0    60   ~ 0
-0V
-$Comp
-L C C?
-U 1 1 506F1B91
-P 4150 1150
-F 0 "C?" H 4200 1250 50  0000 L CNN
-F 1 "100nF" H 4200 1050 50  0000 L CNN
-	1    4150 1150
-	1    0    0    -1
-$EndComp
+	9200 750  4050 750
 Wire Wire Line
 	4150 1350 4150 1700
 Wire Wire Line
 	4150 750  4150 950
-$Comp
-L ZENER D?
-U 1 1 506F1D24
-P 4600 950
-F 0 "D?" H 4600 1050 50  0000 C CNN
-F 1 "20V" H 4600 850 40  0000 C CNN
-	1    4600 950
-	0    -1   -1   0
-$EndComp
-$Comp
-L R R?
-U 1 1 506F1D33
-P 4600 1450
-F 0 "R?" V 4680 1450 50  0000 C CNN
-F 1 "1k" V 4600 1450 50  0000 C CNN
-	1    4600 1450
-	1    0    0    -1
-$EndComp
 Wire Wire Line
 	3100 1700 5300 1700
@@
 	4600 1150 4600 1200
 Connection ~ 4150 750
-$Comp
-L C C?
-U 1 1 506F22D9
-P 4900 1450
-F 0 "C?" H 4950 1550 50  0000 L CNN
-F 1 "47nF" H 4950 1350 50  0000 L CNN
-	1    4900 1450
-	1    0    0    -1
-$EndComp
 Wire Wire Line
 	4900 1700 4900 1650
@@
 Wire Wire Line
 	4900 1200 4900 1250
-$Comp
-L THYRISTOR T?
-U 1 1 506F2A69
-P 5300 1100
-F 0 "T?" H 5200 1200 40  0000 C CNN
-F 1 "THYRISTOR" H 5300 1000 40  0000 C CNN
-	1    5300 1100
-	0    -1   1    0
-$EndComp
 Connection ~ 4900 1200
 Wire Wire Line
@@
 	5300 1700 5300 1300
 Connection ~ 4900 1700
-Text Notes 1150 1750 0    60   ~ 0
-POWER INPUT\n
-Text Notes 3700 1850 0    60   ~ 0
-OVERVOLTAGE CROWBAR
-$Comp
-L DIODE D?
-U 1 1 506F2E41
-P 1650 2450
-F 0 "D?" H 1650 2550 40  0000 C CNN
-F 1 "DIODE" H 1650 2350 40  0000 C CNN
-	1    1650 2450
-	0    -1   -1   0
-$EndComp
 Wire Wire Line
 	1050 2850 3200 2850
@@
 	1600 2250 2050 2250
 Connection ~ 1650 2250
-Text Notes 1350 2650 0    60   ~ 0
-IDIOT\nDIODE
 Connection ~ 5300 750
-Text Notes 14700 1900 0    60   ~ 0
-FLOWMETER CONNECTION
-Text Notes 7450 7950 0    60   ~ 0
-PERIPHERAL CONNECTION CABLE
-Text Notes 11150 7900 0    60   ~ 0
-PERIPHERALS
+$Comp
+L DIL16 P?
+U 1 1 506F3C59
+P 6700 4650
+F 0 "P?" H 6700 5100 60  0000 C CNN
+F 1 "DIL16" V 6700 4650 50  0000 C CNN
+	1    6700 4650
+	1    0    0    -1
+$EndComp
+Text Label 6100 4300 0    60   ~ 0
+GND
+Text Label 6100 4400 0    60   ~ 0
+Vin
+Text Label 6100 4500 0    60   ~ 0
++5V
+Text Label 6100 4600 0    60   ~ 0
+53
+Text Label 6100 4700 0    60   ~ 0
+9
+Text Label 6100 4800 0    60   ~ 0
+7
+Text Label 6100 4900 0    60   ~ 0
+A0
+Text Label 6100 5000 0    60   ~ 0
+A1
+Text Label 7100 4300 0    60   ~ 0
+5
+Text Label 7100 4400 0    60   ~ 0
+37
+Text Label 7100 4500 0    60   ~ 0
+36
+Text Label 7100 4600 0    60   ~ 0
+35
+Text Label 7100 4700 0    60   ~ 0
+34
+Text Label 7100 4800 0    60   ~ 0
+33
+Text Label 7100 4900 0    60   ~ 0
+32
+Text Label 7100 5000 0    60   ~ 0
+31
+Wire Wire Line
+	6100 4300 6350 4300
+Wire Wire Line
+	6350 4400 6100 4400
+Wire Wire Line
+	6100 4500 6350 4500
+Wire Wire Line
+	5550 4600 6350 4600
+Wire Wire Line
+	5550 4700 6350 4700
+Wire Wire Line
+	5550 4800 6350 4800
+Wire Wire Line
+	5550 4900 6350 4900
+Wire Wire Line
+	5550 5000 6350 5000
+Wire Wire Line
+	7050 4300 7300 4300
+Wire Wire Line
+	7050 4400 7300 4400
+Wire Wire Line
+	7050 4500 7300 4500
+Wire Wire Line
+	7050 4600 7300 4600
+Wire Wire Line
+	7050 4700 7300 4700
+Wire Wire Line
+	7050 4800 7300 4800
+Wire Wire Line
+	7050 4900 7300 4900
+Wire Wire Line
+	7050 5000 7300 5000
+Text Label 5550 4600 0    60   ~ 0
+UART1 RX
+Text Label 5550 4700 0    60   ~ 0
+UART1 TX
+Text Label 5550 4800 0    60   ~ 0
+UART2 TX
+Text Label 5550 4900 0    60   ~ 0
+POT_IN
+Text Label 5550 5000 0    60   ~ 0
+BATT_IN
+Text Label 7300 4300 0    60   ~ 0
+KEYSW_IN
+Text Label 7300 4400 0    60   ~ 0
+R1
+Text Label 7300 4500 0    60   ~ 0
+R2
+Text Label 7300 4600 0    60   ~ 0
+R3
+Text Label 7300 4700 0    60   ~ 0
+R4
+Text Label 7300 4800 0    60   ~ 0
+R5
+Text Label 7300 4900 0    60   ~ 0
+R6
+Text Label 7300 5000 0    60   ~ 0
+R7
 $EndSCHEMATC

Commit message: Corrected arduino pin function labels
Parts:
- P?: value DIL16 -> ARDUINO CONNS
Connections:
- net labels removed: R5, R6, R7
Changed lines of the file:
@@
-EESchema Schematic File Version 2  date Fri 05 Oct 2012 19:19:31 BST
+EESchema Schematic File Version 2  date Fri 05 Oct 2012 19:28:29 BST
 LIBS:power
 LIBS:device
@@
 P 6700 4650
 F 0 "P?" H 6700 5100 60  0000 C CNN
-F 1 "DIL16" V 6700 4650 50  0000 C CNN
+F 1 "ARDUINO CONNS" V 6700 4650 50  0000 C CNN
 	1    6700 4650
 	1    0    0    -1
@@
 R4
 Text Label 7300 4800 0    60   ~ 0
-R5
+C1
 Text Label 7300 4900 0    60   ~ 0
-R6
+C2
 Text Label 7300 5000 0    60   ~ 0
-R7
+C3
 $EndSCHEMATC

Commit message: Added keypad pullups and extra labelling
Parts:
- added P?: CONN_2, symbol CONN_2
- added R? (x3): 10k, symbol R
Connections:
- net labels added: FLOWPOT, KEYSW, LCD_DATA, SPK
- net labels removed: DATA, POT_IN, UART2 TX
- wire segments 182 -> 207
Other:
- moved on the sheet: P?
Changed lines of the file:
@@
-EESchema Schematic File Version 2  date Fri 05 Oct 2012 19:28:29 BST
+EESchema Schematic File Version 2  date Fri 05 Oct 2012 19:49:31 BST
 LIBS:power
 LIBS:device
@@
 Text Label 13100 8600 0    60   ~ 0
 0V
-Text Label 11900 8950 0    60   ~ 0
-DATA
-Text Label 11900 9050 0    60   ~ 0
+Text Label 11700 8950 0    60   ~ 0
+LCD_DATA
+Text Label 11700 9050 0    60   ~ 0
 3V3
-Text Label 11900 8850 0    60   ~ 0
+Text Label 11700 8850 0    60   ~ 0
 0V
 Text Label 10150 8250 0    60   ~ 0
@@
 L CONN_14 P?
 U 1 1 50636A9D
-P 5950 7850
-F 0 "P?" V 5920 7850 60  0000 C CNN
-F 1 "CONN_ARD_PERIPHS" V 6030 7850 60  0000 C CNN
-	1    5950 7850
+P 5450 7850
+F 0 "P?" V 5420 7850 60  0000 C CNN
+F 1 "CONN_ARD_PERIPHS" V 5530 7850 60  0000 C CNN
+	1    5450 7850
 	0    -1   -1   0
 $EndComp
@@
 	9400 950  15050 950
 Wire Wire Line
-	6100 8200 6100 9750
-Wire Wire Line
-	5900 8200 5900 9650
-Wire Wire Line
-	5300 8200 5300 10350
-Wire Wire Line
-	5600 8200 5600 8850
-Wire Wire Line
-	5400 8200 5400 8250
-Wire Wire Line
-	6300 8200 6300 9150
-Wire Wire Line
-	6750 8350 6600 8350
-Wire Wire Line
-	6600 8350 6600 8200
+	5600 8200 5600 9750
+Wire Wire Line
+	5400 8200 5400 9650
+Wire Wire Line
+	4800 8200 4800 10350
+Wire Wire Line
+	5100 8200 5100 8850
+Wire Wire Line
+	4900 8200 4900 8250
+Wire Wire Line
+	5800 8200 5800 9150
+Wire Wire Line
+	6100 8350 6750 8350
+Wire Wire Line
+	6100 8350 6100 8200
 Wire Wire Line
 	2050 2050 2050 3200
@@
 	9950 2000 9950 1550
 Wire Wire Line
-	6100 9750 6750 9750
-Wire Wire Line
-	6750 9550 6000 9550
-Wire Wire Line
-	6750 8950 6400 8950
-Wire Wire Line
-	6750 8750 6500 8750
-Wire Wire Line
-	6750 8450 5500 8450
-Wire Wire Line
-	5400 8250 6750 8250
-Wire Wire Line
-	5300 10350 6750 10350
+	5600 9750 6750 9750
+Wire Wire Line
+	5500 9550 6750 9550
+Wire Wire Line
+	5900 8950 6750 8950
+Wire Wire Line
+	6000 8750 6750 8750
+Wire Wire Line
+	5000 8450 6750 8450
+Wire Wire Line
+	4900 8250 6750 8250
+Wire Wire Line
+	4800 10350 6750 10350
 Wire Wire Line
 	8450 2000 8000 2000
@@
 	9850 1450 15050 1450
 Wire Wire Line
-	6750 9950 6200 9950
-Wire Wire Line
-	6750 8650 5700 8650
-Wire Wire Line
-	5600 8850 6750 8850
-Wire Wire Line
-	6300 9150 6750 9150
-Wire Wire Line
-	5900 9650 6750 9650
-Wire Wire Line
-	6750 9850 5800 9850
+	5700 9950 6750 9950
+Wire Wire Line
+	5200 8650 6750 8650
+Wire Wire Line
+	5100 8850 6750 8850
+Wire Wire Line
+	5800 9150 6750 9150
+Wire Wire Line
+	5400 9650 6750 9650
+Wire Wire Line
+	5300 9850 6750 9850
 Wire Wire Line
 	9850 1450 9850 1800
@@
 	13050 8050 13050 8400
 Wire Wire Line
-	13050 8400 13400 8400
-Wire Wire Line
 	9650 9750 13000 9750
 Wire Wire Line
@@
 	13200 9800 15400 9800
 Wire Wire Line
-	6500 8750 6500 8200
-Wire Wire Line
-	6400 8950 6400 8200
-Wire Wire Line
-	5500 8450 5500 8200
-Wire Wire Line
-	5700 8650 5700 8200
-Wire Wire Line
-	5800 9850 5800 8200
-Wire Wire Line
-	6000 9550 6000 8200
-Wire Wire Line
-	6200 9950 6200 8200
+	6000 8750 6000 8200
+Wire Wire Line
+	5900 8950 5900 8200
+Wire Wire Line
+	5000 8450 5000 8200
+Wire Wire Line
+	5200 8650 5200 8200
+Wire Wire Line
+	5300 9850 5300 8200
+Wire Wire Line
+	5500 9550 5500 8200
+Wire Wire Line
+	5700 9950 5700 8200
 Wire Wire Line
 	3100 550  3100 2750
@@
 31
 Wire Wire Line
-	6100 4300 6350 4300
-Wire Wire Line
-	6350 4400 6100 4400
-Wire Wire Line
-	6100 4500 6350 4500
-Wire Wire Line
-	5550 4600 6350 4600
-Wire Wire Line
-	5550 4700 6350 4700
+	4250 4300 6350 4300
+Wire Wire Line
+	4350 4400 6350 4400
+Wire Wire Line
+	5800 4500 6350 4500
+Wire Wire Line
+	4850 4600 6350 4600
 Wire Wire Line
 	5550 4800 6350 4800
@@
 	5550 4900 6350 4900
 Wire Wire Line
-	5550 5000 6350 5000
-Wire Wire Line
-	7050 4300 7300 4300
-Wire Wire Line
-	7050 4400 7300 4400
-Wire Wire Line
-	7050 4500 7300 4500
-Wire Wire Line
-	7050 4600 7300 4600
-Wire Wire Line
-	7050 4700 7300 4700
-Wire Wire Line
-	7050 4800 7300 4800
-Wire Wire Line
-	7050 4900 7300 4900
-Wire Wire Line
-	7050 5000 7300 5000
+	5350 5000 6350 5000
+Wire Wire Line
+	7050 4300 7800 4300
+Wire Wire Line
+	7050 4400 7700 4400
+Wire Wire Line
+	7050 4500 7650 4500
+Wire Wire Line
+	7050 4600 7600 4600
+Wire Wire Line
+	7050 4700 7550 4700
+Wire Wire Line
+	7050 4800 7950 4800
+Wire Wire Line
+	7050 4900 8150 4900
+Wire Wire Line
+	7050 5000 8350 5000
 Text Label 5550 4600 0    60   ~ 0
 UART1 RX
@@
 UART1 TX
 Text Label 5550 4800 0    60   ~ 0
-UART2 TX
+LCD_DATA
 Text Label 5550 4900 0    60   ~ 0
-POT_IN
+FLOWPOT
 Text Label 5550 5000 0    60   ~ 0
 BATT_IN
@@
 Text Label 7300 5000 0    60   ~ 0
 C3
+Wire Wire Line
+	5800 4500 5800 3950
+Wire Wire Line
+	5800 3950 7900 3950
+Wire Wire Line
+	7550 4700 7550 5250
+Wire Wire Line
+	7600 4600 7600 5250
+Wire Wire Line
+	7650 4500 7650 5250
+Wire Wire Line
+	7700 4400 7700 5250
+Wire Wire Line
+	7950 4800 7950 4700
+$Comp
+L R R?
+U 1 1 506F6F28
+P 7950 4450
+F 0 "R?" V 8030 4450 50  0000 C CNN
+F 1 "10k" V 7950 4450 50  0000 C CNN
+	1    7950 4450
+	1    0    0    -1
+$EndComp
+$Comp
+L R R?
+U 1 1 506F6F37
+P 8150 4450
+F 0 "R?" V 8230 4450 50  0000 C CNN
+F 1 "10k" V 8150 4450 50  0000 C CNN
+	1    8150 4450
+	1    0    0    -1
+$EndComp
+$Comp
+L R R?
+U 1 1 506F6F46
+P 8350 4450
+F 0 "R?" V 8430 4450 50  0000 C CNN
+F 1 "10k" V 8350 4450 50  0000 C CNN
+	1    8350 4450
+	1    0    0    -1
+$EndComp
+Connection ~ 7950 4200
+Connection ~ 8150 4200
+Wire Wire Line
+	8150 4900 8150 4700
+Wire Wire Line
+	8350 5000 8350 4700
+Wire Wire Line
+	7800 4300 7800 3800
+Wire Wire Line
+	7900 3950 7900 4200
+Wire Wire Line
+	7900 4200 8350 4200
+Wire Wire Line
+	5350 4400 5350 5000
+Text Label 13100 8400 0    60   ~ 0
+SPK
+Wire Wire Line
+	13050 8400 13400 8400
+Text Label 10250 8500 0    60   ~ 0
+FLOWPOT
+Text Label 9950 10350 0    60   ~ 0
+KEYSW
+Wire Wire Line
+	4850 4600 4850 2350
+Wire Wire Line
+	4850 2350 6400 2350
+Wire Wire Line
+	6400 2350 6400 1800
+Wire Wire Line
+	6400 1800 7200 1800
+Wire Wire Line
+	4750 4700 4750 2250
+Wire Wire Line
+	4750 2250 6300 2250
+Wire Wire Line
+	6300 2250 6300 1700
+Wire Wire Line
+	6300 1700 7200 1700
+Wire Wire Line
+	4750 4700 6350 4700
+$Comp
+L CONN_2 P?
+U 1 1 506F9349
+P 3050 3300
+F 0 "P?" V 3000 3300 40  0000 C CNN
+F 1 "CONN_2" V 3100 3300 40  0000 C CNN
+	1    3050 3300
+	-1   0    0    1
+$EndComp
+Wire Wire Line
+	3400 3400 4250 3400
+Wire Wire Line
+	4250 3400 4250 4300
+Wire Wire Line
+	3400 3200 4350 3200
+Wire Wire Line
+	4350 3200 4350 4400
+Connection ~ 5350 4400
+Text Label 6300 8250 0    60   ~ 0
++5V
+Text Label 6300 8350 0    60   ~ 0
+C1
+Text Label 6300 8450 0    60   ~ 0
+FLOWPOT
+Text Label 6300 8650 0    60   ~ 0
+SPK
+Text Label 6300 8750 0    60   ~ 0
+R2
+Text Label 6300 8850 0    60   ~ 0
+0V
+Text Label 6300 8950 0    60   ~ 0
+R3
+Text Label 6300 9150 0    60   ~ 0
+C2
+Text Label 6300 9550 0    60   ~ 0
+C3
+Text Label 6300 9650 0    60   ~ 0
+LCD_DATA
+Text Label 6300 9750 0    60   ~ 0
+R1
+Text Label 6300 9850 0    60   ~ 0
+3V3
+Text Label 6300 9950 0    60   ~ 0
+R4
+Text Label 6300 10350 0    60   ~ 0
+KEYSW
 $EndSCHEMATC

Commit message: Added SPK pin to arduino IO
Parts:
- removed P?: ARDUINO CONNS, symbol DIL16
- added P?: ARDUINO CONNS, symbol CONN_8
- added P?: ARDUINO CONNS, symbol CONN_9
Connections:
- net labels added: 30
- wire segments 207 -> 209
Other:
- moved on the sheet: R?
Changed lines of the file:
@@
-EESchema Schematic File Version 2  date Fri 05 Oct 2012 19:49:31 BST
+EESchema Schematic File Version 2  date Fri 05 Oct 2012 19:54:39 BST
 LIBS:power
 LIBS:device
@@
 Connection ~ 1650 2250
 Connection ~ 5300 750
-$Comp
-L DIL16 P?
-U 1 1 506F3C59
-P 6700 4650
-F 0 "P?" H 6700 5100 60  0000 C CNN
-F 1 "ARDUINO CONNS" V 6700 4650 50  0000 C CNN
-	1    6700 4650
-	1    0    0    -1
-$EndComp
 Text Label 6100 4300 0    60   ~ 0
 GND
@@
 Text Label 6100 5000 0    60   ~ 0
 A1
-Text Label 7100 4300 0    60   ~ 0
+Text Label 7300 4300 0    60   ~ 0
 5
-Text Label 7100 4400 0    60   ~ 0
+Text Label 7300 4400 0    60   ~ 0
 37
-Text Label 7100 4500 0    60   ~ 0
+Text Label 7300 4500 0    60   ~ 0
 36
-Text Label 7100 4600 0    60   ~ 0
+Text Label 7300 4600 0    60   ~ 0
 35
-Text Label 7100 4700 0    60   ~ 0
+Text Label 7300 4700 0    60   ~ 0
 34
-Text Label 7100 4800 0    60   ~ 0
+Text Label 7300 4800 0    60   ~ 0
 33
-Text Label 7100 4900 0    60   ~ 0
+Text Label 7300 4900 0    60   ~ 0
 32
-Text Label 7100 5000 0    60   ~ 0
+Text Label 7300 5000 0    60   ~ 0
 31
 Wire Wire Line
@@
 	5350 5000 6350 5000
 Wire Wire Line
-	7050 4300 7800 4300
-Wire Wire Line
-	7050 4400 7700 4400
-Wire Wire Line
-	7050 4500 7650 4500
-Wire Wire Line
-	7050 4600 7600 4600
-Wire Wire Line
-	7050 4700 7550 4700
-Wire Wire Line
-	7050 4800 7950 4800
-Wire Wire Line
-	7050 4900 8150 4900
-Wire Wire Line
-	7050 5000 8350 5000
+	7250 4300 8000 4300
+Wire Wire Line
+	7250 4400 7900 4400
+Wire Wire Line
+	7250 4500 7850 4500
+Wire Wire Line
+	7250 4600 7800 4600
+Wire Wire Line
+	7250 4700 7750 4700
+Wire Wire Line
+	7250 4800 8150 4800
+Wire Wire Line
+	7250 4900 8350 4900
+Wire Wire Line
+	7250 5000 8550 5000
 Text Label 5550 4600 0    60   ~ 0
 UART1 RX
@@
 Text Label 5550 5000 0    60   ~ 0
 BATT_IN
-Text Label 7300 4300 0    60   ~ 0
+Text Label 7500 4300 0    60   ~ 0
 KEYSW_IN
-Text Label 7300 4400 0    60   ~ 0
+Text Label 7500 4400 0    60   ~ 0
 R1
-Text Label 7300 4500 0    60   ~ 0
+Text Label 7500 4500 0    60   ~ 0
 R2
-Text Label 7300 4600 0    60   ~ 0
+Text Label 7500 4600 0    60   ~ 0
 R3
-Text Label 7300 4700 0    60   ~ 0
+Text Label 7500 4700 0    60   ~ 0
 R4
-Text Label 7300 4800 0    60   ~ 0
+Text Label 7500 4800 0    60   ~ 0
 C1
-Text Label 7300 4900 0    60   ~ 0
+Text Label 7500 4900 0    60   ~ 0
 C2
-Text Label 7300 5000 0    60   ~ 0
+Text Label 7500 5000 0    60   ~ 0
 C3
 Wire Wire Line
 	5800 4500 5800 3950
 Wire Wire Line
-	5800 3950 7900 3950
-Wire Wire Line
-	7550 4700 7550 5250
-Wire Wire Line
-	7600 4600 7600 5250
-Wire Wire Line
-	7650 4500 7650 5250
-Wire Wire Line
-	7700 4400 7700 5250
-Wire Wire Line
-	7950 4800 7950 4700
+	5800 3950 8100 3950
+Wire Wire Line
+	7750 4700 7750 5250
+Wire Wire Line
+	7800 4600 7800 5250
+Wire Wire Line
+	7850 4500 7850 5250
+Wire Wire Line
+	7900 4400 7900 5250
+Wire Wire Line
+	8150 4800 8150 4700
 $Comp
 L R R?
 U 1 1 506F6F28
-P 7950 4450
-F 0 "R?" V 8030 4450 50  0000 C CNN
-F 1 "10k" V 7950 4450 50  0000 C CNN
-	1    7950 4450
-	1    0    0    -1
-$EndComp
-$Comp
-L R R?
-U 1 1 506F6F37
 P 8150 4450
 F 0 "R?" V 8230 4450 50  0000 C CNN
@@
 $Comp
 L R R?
-U 1 1 506F6F46
+U 1 1 506F6F37
 P 8350 4450
 F 0 "R?" V 8430 4450 50  0000 C CNN
@@
 	1    0    0    -1
 $EndComp
-Connection ~ 7950 4200
+$Comp
+L R R?
+U 1 1 506F6F46
+P 8550 4450
+F 0 "R?" V 8630 4450 50  0000 C CNN
+F 1 "10k" V 8550 4450 50  0000 C CNN
+	1    8550 4450
+	1    0    0    -1
+$EndComp
 Connection ~ 8150 4200
-Wire Wire Line
-	8150 4900 8150 4700
-Wire Wire Line
-	8350 5000 8350 4700
-Wire Wire Line
-	7800 4300 7800 3800
-Wire Wire Line
-	7900 3950 7900 4200
-Wire Wire Line
-	7900 4200 8350 4200
+Connection ~ 8350 4200
+Wire Wire Line
+	8350 4900 8350 4700
+Wire Wire Line
+	8550 5000 8550 4700
+Wire Wire Line
+	8000 4300 8000 3800
+Wire Wire Line
+	8100 3950 8100 4200
+Wire Wire Line
+	8100 4200 8550 4200
 Wire Wire Line
 	5350 4400 5350 5000
@@
 Text Label 6300 10350 0    60   ~ 0
 KEYSW
+$Comp
+L CONN_8 P?
+U 1 1 506FB0F8
+P 6700 4650
+F 0 "P?" V 6650 4650 60  0000 C CNN
+F 1 "ARDUINO CONNS" V 6750 4650 60  0000 C CNN
+	1    6700 4650
+	1    0    0    -1
+$EndComp
+$Comp
+L CONN_9 P?
+U 1 1 506FB107
+P 6900 4700
+F 0 "P?" V 6850 4700 60  0000 C CNN
+F 1 "ARDUINO CONNS" V 6950 4700 60  0000 C CNN
+	1    6900 4700
+	-1   0    0    -1
+$EndComp
+Wire Wire Line
+	7250 5100 8550 5100
+Wire Wire Line
+	8550 5100 8550 5350
+Text Label 7300 5100 0    60   ~ 0
+30
+Text Label 7500 5100 0    60   ~ 0
+SPK
 $EndSCHEMATC
